File: pcb/albert.kicad_sch (KiCad schematic)
At the start: 72 parts, among them IC1 STM32U585CIUx, IC2 ADAU1466, J1 USB_C_Receptacle_USB2.0, J2 Conn_01x03_Pin, Q1 STD2805, SW1 SW_SPDT, U1 LT8640A, U2 STPD01, U3 NUP4202, U4 AQV252G2SX, Y1 12M288

Commit message: Added hall sensor for BLDC
Parts:
- added C45: 100n, symbol Device:C_Feedthrough
- added U6: MLX90363, Package_SO:SOIC-8_3.9x4.9mm_P1.27mm, symbol albert:MLX90363
- R8: value 47 -> 220
Connections:
- net +3.3V: now also C45.1
- net GND1: now also C45.2, U6.3 (TEST), U6.8 (VSS)
- net USB_CC1: now also IC1.38 (PA15)
- net USB_CC2: now also IC1.28 (PB15)
- net VBUS_EN: now also IC1.5 (PH0)
- net VBUS_SW: now also IC1.6 (PH1)
- net USB_SDP: now reaches IC1.31 (PA10)
- net USB_SDN: now reaches IC1.32 (PA11)
- new net: C45.3, U6.1 (VDD), U6.7 (VDEC)
- new net HALL_*SS: U6.5 (*SS)
- new net SPI_MISO: U6.2 (MISO)
- new net SPI_MOSI: U6.6 (MOSI)
- new net SPI_SCK: U6.4 (SCK)
Other:
- note added: "Knob Hall Sensor"
- moved on the sheet: C38, C39, C40, C41

Commit message: Updated power supply solution
Parts:
- removed C10, C27: 100n, symbol Device:C
- removed C19, C20, C28, C29, C30, C31, C36, C45: 100n, symbol Device:C_Feedthrough
- removed C25, C38, C40: 10u, symbol Device:C
- removed C42: 22p, symbol Device:C
- removed Q1: STD2805, symbol Device:Q_PNP_BCE
- removed U1: LT8640A, albert:LT8640, symbol albert:LT8640A
- removed U6: MLX90363, Package_SO:SOIC-8_3.9x4.9mm_P1.27mm, symbol albert:MLX90363
- added C10, C25, C27, C38, C40, C42, C44, C46, C52, C53, C54, C75, C77: 100n, symbol Device:C_Feedthrough
- added C19, C48, C59, C63, C68, C78: 100n, symbol Device:C
- added C20: C, symbol Device:C
- added C28: 150p, symbol Device:C
- added C29, C30: 22p, symbol Device:C
- added C31, C50: 5n6, symbol Device:C
- added C36, C55, C56, C57, C58, C60, C67, C76: 10u, symbol Device:C
- added C45, C71, C72, C73: 4u7, symbol Device:C
- added C47: 100u, symbol Device:C
- added C49: 220n, symbol Device:C
- added C51: 10n, symbol Device:C
- added C61, C62: 470n, symbol Device:C
- added C64: 47p, symbol Device:C
- added C65, C66, C79, C80, C81, C82: 22u, symbol Device:C
- added D4, D5: 1N4148, Diode_THT:D_DO-35_SOD27_P7.62mm_Horizontal, symbol Diode:1N4148
- added D6, D7, D8, D9: D, symbol Device:D
- added J3: Conn_01x03_Pin, symbol Connector:Conn_01x03_Pin
- added L3: 6u8, symbol Device:L
- added L4: 10u, symbol Device:L
- added R13: 100, symbol Device:R
- added R14, R18, R28: 10k, symbol Device:R
- added R15, R16, R17: 22m, symbol Device:R
- added R19: 15k, symbol Device:R
- added R20, R23: 24k, symbol Device:R
- added R21: 51k, symbol Device:R
- added R22: 12k, symbol Device:R
- added R24: 499, symbol Device:R
- added R25: 33k2, symbol Device:R
- added R26: 453k, symbol Device:R
- added R27: 49k9, symbol Device:R
- added R29: 20k, symbol Device:R
- added R30: 620m, symbol Device:R
- added R31: 75k, symbol Device:R
- added R32: 9k1, symbol Device:R
- added TH1, TH2: Thermistor, symbol Device:Thermistor
- added TR1: TRANSF6, symbol Transformer:TRANSF6
- added U1, U12, U17: AP63357, albert:VFDFN3020-13, symbol albert:AP63357
- added U10, U8, U9: INA180A2, Package_TO_SOT_SMD:SOT-23-5, symbol Amplifier_Current:INA180A2
- added U11: SN6507, Package_SO:HVSSOP-10-1EP_3x3mm_P0.5mm_EP1.57x1.88mm_ThermalVias, symbol albert:SN6507
- added U14: LT3042xMSE, Package_SO:MSOP-10-1EP_3x3mm_P0.5mm_EP1.68x1.88mm, symbol Regulator_Linear:LT3042xMSE
- added U16: ADUM340E, Package_SO:SOIC-16W_7.5x10.3mm_P1.27mm, symbol albert:ADUM340E
- added U5: MLX90395, Package_DFN_QFN:QFN-16-1EP_3x3mm_P0.5mm_EP1.7x1.7mm, symbol albert:MLX90395
- added U6: L6230, Package_SO:HSOP-36-1EP_11.0x15.9mm_P0.65mm_SlugDown_ThermalVias, symbol albert:L6230
- added U7: TPS7A87, Package_DFN_QFN:WQFN-24-1EP_4x4mm_P0.5mm_EP2.6x2.6mm_ThermalVias, symbol albert:TPS7A87
- C1: value 1u -> 10u
- C2: value 10n -> 100n
- C24: value C -> 10u
- C3: value 1u -> 47p
- C4: value 1u -> 22u
- C43: value 22p -> 10u
- C5: value 4u7 -> 22u
- C6: value 100n -> 1u
- C7: value 10p -> 1u
- C8: value 100u -> 10n
- C9: value 10u -> 10n
- L1: value 1u -> 6u8
- R1: value 18k2 -> 51k
- R10: value 10k -> 4k3
- R11: value 100 -> 10k
- R12: value 1k -> 75k
- R2: value 1M -> 12k
- R3: value 412k -> 10k
- R4: value 620m -> 10k
Connections:
- net DSP_EN is gone; now on net VDD_OK: IC2.24 (~{RESET})
- net +24V: now also C1.1, C56.1, C76.1, TR1.2, TR1.3, U1.1 (VIN), U1.2 (EN), U11.3 (VCC), U11.4 (EN/UVLO), U17.1 (VIN), U17.2 (EN); no longer C3.1, C4.1, C5.1
- net +3.3V: now also C23.3, C24.1, C37.3, R12.1, C10.1, C25.3, C28.1, C31.1, C38.3, C40.3, C42.3, C58.1, C59.1, C77.3, R14.2, U7.11 (OUT2), U7.12 (OUT2); no longer C32.3, C33.3, C34.3, C35.3, C7.1, L1.2, R12.2, R2.1
- net +3.3VA: now also C43.1, C27.3, C44.3, C46.3, C52.1, C53.1, C54.1, C55.1, C60.1, C68.1; no longer C23.3, C37.3, C9.1
- net GND1: now also C1.2, C43.2, C6.2, C7.2, IC2.3 (VDRIVE), R11.1, R2.2, C10.2, C19.1, C20.2, C25.2, C27.2, C29.1, C30.1, C36.2, C38.2, C40.2, C42.2, C44.2, C45.2, C46.2, C47.2, C48.2, C50.2, C52.2, C53.2, C54.2, C55.2, C56.2, C57.2, C58.2, C59.2, C68.2, C76.2, C79.2, C80.2, C81.2, C82.2, R19.2, R20.2, R23.2, R29.2, R30.1, R32.2, U1.4 (COMP), U1.8 (GND), U10.2 (GND), U11.11 (GND), U11.2 (GND), U11.7 (CLK), U11.9 (GND), U17.4 (COMP), U17.8 (GND), U5.10 (NC), U5.11 (NC), U5.12 (NC), U5.13 (VSS), U5.14 (NC), U5.16 (NC), U5.4 (NC), U5.8 (NC), U5.9 (NC), U6.1 (GND), U6.12 (SENSE1), U6.18 (GND), U6.19 (GND), U6.25 (SENSE3), U6.36 (GND), U6.8 (SENSE2), U7.13 (GND), U7.25 (GND), U7.3 (GND), U8.2 (GND), U9.2 (GND); no longer C1.1, C2.1, C3.2, C43.1, C8.2, R1.1, R10.1, R3.2, R4.2
- net HALL_*SS: now also IC1.39 (PB3), U5.2 (*SS)
- net SAI_FS: now also IC1.30 (PA9)
- net SAI_SCK: now also IC1.29 (PA8)
- net SAI_SD: now also IC1.31 (PA10)
- net SPI_MISO: now also IC1.16 (PA6), U5.6 (MISO)
- net SPI_MOSI: now also IC1.17 (PA7), U5.5 (MOSI)
- net SPI_SCK: now also IC1.15 (PA5), U5.3 (SCK)
- net TDM_FS: now also U16.4 (VIB)
- net TDM_SCK: now also U16.3 (VIA)
- net TDM_SD: now also U16.5 (VIC)
- net USB_SDP: now also IC1.33 (PA12); no longer IC1.31 (PA10)
- net at IC1.24 (VDD): now also C22.1
- net at C6.1: now also U7.19 (NR/SS1)
- net at L1.1: now also C2.2, U1.9 (SW); no longer C6.2
- net at IC2.35 (DVDD): now also C33.1
- net at IC2.20 (DVDD): now also C32.1
- net at IC2.15 (PVDD): now also C46.1; no longer C37.1
- net at IC2.16 (PLLFILT): now also R10.2, C28.2
- net at IC2.18 (IOVDD): now also C38.1; no longer C33.1
- net at IC2.2 (IOVDD): now also C37.1; no longer C32.1
- net at IC2.21 (XTALIN/MCLK), Y1.3: now also C29.2
- net at IC2.22 (XTALOUT): now also R13.2; no longer R11.2
- net at IC2.34 (SELFBOOT): now also R11.2; no longer R10.2
- net at IC2.38 (IOVDD): now also C40.1; no longer C34.1
- net at IC2.53 (DVDD): now also C34.1
- net at IC2.56 (IOVDD): now also C42.1; no longer C35.1
- net at IC2.7 (AVDD): now also C44.1
- net at IC2.71 (DVDD): now also C35.1
- net at IC1.36 (VDD): now also C23.1; no longer C21.1
- net at R1.2: now also C3.2, R2.1, U1.3 (FB)
- net at IC1.9 (VDDA): now also C27.1; no longer C23.1
- net at C9.2: now also R28.2, R29.1, U7.16 (FB1); no longer R4.1
- net at IC1.1 (VBAT): now also C21.1
- net BLDC_I1: now reaches IC1.10 (PA0)
- net BLDC_I1: now also U8.1
- net BLDC_I2: now reaches IC1.11 (PA1)
- net BLDC_I2: now also U9.1
- net BLDC_I3: now reaches IC1.12 (PA2)
- net BLDC_I3: now also U10.1
- net BLDC_OK: now reaches IC1.14 (PA4)
- net BLDC_OK: now also C50.1, R14.1, U17.5 (PG), U6.22 (DIAG/EN)
- net at IC1.22 (VCAP): now also C20.1; no longer C24.1
- net MUTE: now reaches IC1.34 (PA13)
- net MUTE: now also U16.6 (VID)
- net BLDC_IN1: now reaches IC1.40 (PB4)
- net BLDC_IN1: now also U6.9 (IN1)
- net BLDC_EN1: now reaches IC1.41 (PB5)
- net BLDC_EN1: now also U6.10 (EN1)
- net BLDC_IN2: now reaches IC1.42 (PB6)
- net BLDC_IN2: now also U6.26 (IN2)
- net BLDC_EN2: now reaches IC1.43 (PB7)
- net BLDC_EN2: now also U6.27 (EN2)
- net BLDC_IN3: now reaches IC1.45 (PB8)
- net BLDC_IN3: now also U6.11 (IN3)
- net BLDC_EN3: now reaches IC1.46 (PB9)
- net BLDC_EN3: now also U6.29 (EN3)
- net at IC1.48 (VDD): now also C25.1; no longer C22.1
- net VDD_OK: now reaches IC1.7 (NRST)
- net VDD_OK: now also C19.2, U7.17 (PG1), U7.9 (PG2)
- net MCLK: no longer names the net of IC2.23 (CLKOUT)
- new net: C31.2, R10.1
- new net: C64.2, R21.2, R22.1, U12.3 (FB)
- new net: C77.1, U16.1 (VDD1)
- new net: C75.1, U16.16 (VDD2)
- new net: R16.1, U6.5 (OUT2), U9.3 (+)
- new net: J3.2 (Pin_2), R16.2, U9.4 (-)
- new net: C53.3, U9.5 (V+)
- new net: C45.1, R20.1, U11.8 (SS/ILIM)
- new net: C10.3, U5.15 (VDD)
- new net: C61.1, D6.1 (K), D8.1 (K), TH1.1
- new net: D7.1 (K), D8.2 (A), TR1.5
- new net: C72.1, R25.1, U14.7 (SET)
- new net: C3.1, C4.1, C5.1, L1.2, R1.1, R4.2, U7.1 (IN1), U7.18 (SS_CTRL1), U7.2 (IN1), U7.4 (IN2), U7.5 (IN1), U7.8 (SS_CTRL2)
- new net: C8.2, R12.2, R23.1, U7.10 (FB2)
- new net: R4.1, U1.5 (PG), U7.20 (EN1), U7.6 (EN2)
- new net: C7.1, U7.7 (NR/SS2)
- new net: C62.2, D7.2 (A), D9.2 (A), TH2.1
- new net: R26.2, R27.1, U14.6 (PGFB)
- new net: R24.1, U14.5 (ILIM)
- new net: C2.1, U1.6 (BST)
- new net: C51.1, D4.1 (K), D5.2 (A)
- new net: R15.1, U6.15 (OUT1), U8.3 (+)
- new net: J3.1 (Pin_1), R15.2, U8.4 (-)
- new net: TR1.1, U11.1 (SW1)
- new net: TR1.4, U11.10 (SW2)
- new net: D6.2 (A), D9.1 (K), TR1.8
- new net: R17.1, U10.3 (+), U6.32 (OUT3)
- new net: J3.3 (Pin_3), R17.2, U10.4 (-)
- new net: C54.3, U10.5 (V+)
- new net: C51.2, U6.7 (VCP)
- new net: C52.3, U8.5 (V+)
- new net: C60.2, R30.2
- new net: C63.2, L3.1, U12.9 (SW)
- new net: R19.1, U11.6 (SR)
- new net: C78.1, U17.6 (BST)
- new net: C78.2, L4.1, U17.9 (SW)
- new net: C49.2, D5.1 (K), U6.30 (VBOOT)
- new net: R31.2, R32.1, U17.3 (FB)
- new net: C63.1, U12.6 (BST)
- new net: C30.2, R13.1, Y1.1
- new net +15V: C67.1, TH1.2, U12.1 (VIN), U12.2 (EN)
- new net +1V2: C32.3, C33.3, C34.3, C35.3, C36.1, C57.1, C9.1, R28.1, U7.14 (OUT1), U7.15 (OUT1)
- new net -15V: TH2.2
- new net BLDC_VDD: C47.1, C48.1, C49.1, C79.1, C80.1, C81.1, C82.1, D4.2 (A), L4.2, R31.1, U6.33 (VSB), U6.4 (VSA)
- new net DAC_AVDD: C73.1, R26.1, U14.10 (OUT), U14.9 (OUTS)
- new net DAC_EN: R18.2, U14.4 (PG), U16.10 (VE2)
- new net DAC_FS: U16.13 (VOB)
- new net DAC_IOVDD: C75.3, R18.1
- new net DAC_MUTE: U16.11 (VOD)
- new net DAC_SCK: U16.14 (VOA)
- new net DAC_SD: U16.12 (VOC)
- new net GND: C77.2, U16.2 (GND1), U16.8 (GND1)
- new net GND2: C61.2, C62.1, C65.2, C66.2, C67.2, C71.2, C72.2, C73.2, C75.2, R22.2, R24.2, R25.2, R27.2, TR1.6, TR1.7, U12.4 (COMP), U12.8 (GND), U14.11 (GND), U14.8 (GND), U16.15 (GND2), U16.9 (GND2)
- new net VIR: C64.1, C65.1, C66.1, C71.1, L3.2, R21.1, R3.2, U14.1 (IN), U14.2 (IN)
- new net VIR_OK: R3.1, U12.5 (PG), U14.3 (EN/UV)
Other:
- note added: "BLDC Motor Driver (FOC)"
- note added: "BLDC Power Supply (7v4)"
- note added: "Control Knob"
- note added: "Digital Processing"
- note added: "Digital Processing Power Supply"
- note added: "Inputs"
- note added: "Isolated DC Power Supply"
- note added: "Isolated Regulator"
- note added: "MCU"
- note added: "Power Input"
- note removed: "Main 3V3 Supply"
- moved on the sheet: C11, C12, C13, C14, C15, C16, C17, C18, D1, D2, D3, J1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

Commit message: Last version before MCU overhaul
Parts:
- removed C15: 47u, symbol Device:C
- removed C52, C75, C77: 100n, symbol Device:C_Feedthrough
- removed C55: 10u, symbol Device:C
- removed D1, D6, D7, D8, D9: D, symbol Device:D
- removed D2: SMAJ24A, Diode_SMD:D_SMA, symbol Diode:SMAJ24A
- removed J2: Conn_01x03_Pin, Connector_Molex:Molex_Micro-Fit_3.0_43650-0300_1x03_P3.00mm_Horizontal, symbol Connector:Conn_01x03_Pin
- removed L3: 6u8, symbol Device:L
- removed TH1, TH2: Thermistor, symbol Device:Thermistor
- removed TR1: TRANSF6, symbol Transformer:TRANSF6
- removed U11: SN6507, Package_SO:HVSSOP-10-1EP_3x3mm_P0.5mm_EP1.57x1.88mm_ThermalVias, symbol albert:SN6507
- removed U12: AP63357, albert:VFDFN3020-13, symbol albert:AP63357
- removed U14: LT3042xMSE, Package_SO:MSOP-10-1EP_3x3mm_P0.5mm_EP1.68x1.88mm, symbol Regulator_Linear:LT3042xMSE
- removed U16: ADUM340E, Package_SO:SOIC-16W_7.5x10.3mm_P1.27mm, symbol albert:ADUM340E
- removed U2: STPD01, Package_DFN_QFN:QFN-24-1EP_3x4mm_P0.4mm_EP1.65x2.65mm_ThermalVias, symbol albert:STPD01
- removed U3: NUP4202, Package_TO_SOT_SMD:SOT-363_SC-70-6, symbol Power_Protection:NUP4202
- removed U6: L6230, Package_SO:HSOP-36-1EP_11.0x15.9mm_P0.65mm_SlugDown_ThermalVias, symbol albert:L6230
- removed Y1: 12M288, symbol Device:Crystal_GND24
- added C106, C52, C69, C70, C89, C90, C91, C92, C93, C94: 10u, symbol Device:C
- added C15, C55: 100n, symbol Device:C_Feedthrough
- added C74: 47n, symbol Device:C
- added C75: 220p, symbol Device:C
- added C77: 100n, symbol Device:C
- added C83, C84, C95, C96, C97: 22u, symbol Device:C
- added C85, C86: 1u, symbol Device:C
- added C87, C88: 10n, symbol Device:C
- added D1: SMAJ20A, Diode_SMD:D_SMA, symbol Diode:SMAJ20A
- added D2, D6: D_Schottky, symbol Device:D_Schottky
- added IC3: L6234, DIP880W50P254L2480H510Q20N, symbol albert:L6234
- added J2: PWR, symbol Connector:Screw_Terminal_01x03
- added J4: NSJ12HF-1, Connector_Audio:Jack_6.35mm_Neutrik_NSJ12HF-1_Horizontal, symbol Connector_Audio:NSJ12HF-1
- added R33: 220, symbol Device:R
- added R36: 75k, symbol Device:R
- added R37: 24k, symbol Device:R
- added R38: 10k, symbol Device:R
- added R39: 20k, symbol Device:R
- added U11: LT3042xMSE, Package_SO:MSOP-10-1EP_3x3mm_P0.5mm_EP1.68x1.88mm, symbol Regulator_Linear:LT3042xMSE
- added U12: LTC3265, Package_DFN_QFN:DFN-18-1EP_3x5mm_P0.5mm_EP1.66x4.4mm, symbol albert:LTC3265
- added U13: STM32H723VGHx, Package_BGA:TFBGA-100_8x8mm_Layout10x10_P0.8mm, symbol MCU_ST_STM32H7:STM32H723VGHx
- added U14: 74LVC1G00, symbol 74xGxx:74LVC1G00
- added U15: TPS7A87, Package_DFN_QFN:WQFN-24-1EP_4x4mm_P0.5mm_EP2.6x2.6mm_ThermalVias, symbol albert:TPS7A87
- added U2: USB3343, Package_DFN_QFN:QFN-24-1EP_4x4mm_P0.5mm_EP2.6x2.6mm, symbol Interface_USB:USB3343
- added U3: PTPS55289RYQR, RYQ0021A-MFG, symbol albert:PTPS55289RYQR
- added Y2: 12M, symbol Device:Crystal_GND24
- C11: value 47u -> 22u
- C12: value 1u -> 22u
- C13: value 1u -> 10u
- C16: value 47u -> 10u
- C17: value 22u -> 1u
- C18: value 10n -> 1u
- C29: value 22p -> 10n
- C30: value 22p -> 10u
- C45, C71: value 4u7 -> 10u
- C50: value 5n6 -> 1u
- C56, L2: value 10u -> 4u7
- C61: value 470n -> 10u
- C62: value 470n -> 1u
- C63: value 100n -> 10u
- C64: value 47p -> 1u
- C65, C66: value 22u -> 100n
- C72, C73: value 4u7 -> 100n
- C76: value 10u -> 22u
- R1: value 51k -> 10k
- R13: value 100 -> 2k67
- R14: value 10k -> 10m
- R18: value 10k -> 52k3
- R19: value 15k -> 499
- R2: value 12k -> 43k
- R20: value 24k -> 33k2
- R21: value 51k -> 52k3
- R22: value 12k -> 604k
- R24: value 499 -> 13k7
- R25: value 33k2 -> 14k3
- R26: value 453k -> 100k
- R27: value 49k9 -> 10k
- R3: value 10k -> 604k
- R4: value 10k -> 8k2
- R5: value 24k -> 1M78
- R6: value 25m -> 100k
- R7: value 10k -> 48k7
- R8: value 220 -> 8k06
Connections:
- net +24V: now also C12.1, C14.1, R5.1, J2.3 (Pin_3), U3.7 (VIN); no longer C1.1, C56.1, U1.1 (VIN), U1.2 (EN)
- net +3.3V: now also C13.2, C19.1, C106.1, C15.3; no longer R14.2
- net +3.3VA: now also C52.1, C55.1
- net BLDC_EN1: now also IC3.3 (EN1)
- net BLDC_EN2: now also IC3.18 (EN2)
- net BLDC_EN3: now also IC3.8 (EN3)
- net BLDC_I1: now also U13.G2 (PA0); no longer IC1.10 (PA0)
- net BLDC_I2: now also U13.H2 (PA1); no longer IC1.11 (PA1)
- net BLDC_I3: now also U13.G3 (PA4); no longer IC1.12 (PA2)
- net BLDC_IN1: now also IC3.2 (IN1)
- net BLDC_IN2: now also IC3.19 (IN2)
- net BLDC_IN3: now also IC3.9 (IN3)
- net BLDC_OK: no longer C50.1, R14.1
- net BLDC_VDD: now also C49.2, IC3.4 (VS), IC3.7 (VS); no longer C49.1
- net DAC_AVDD: now also C61.1, R24.1, U11.10 (OUT), U11.9 (OUTS); no longer C73.1, R26.1
- net DAC_EN: now also R27.1, U11.4 (PG), U15.17 (PG1), U15.9 (PG2); no longer R18.2
- net DAC_IOVDD: now also R27.2, C87.1, C90.1, R36.1, U14.5 (VCC), U15.11 (OUT2), U15.12 (OUT2); no longer R18.1
- net I2C_SCL: now also U13.B4 (PB8), U3.3 (SCL)
- net I2C_SDA: now also U13.A4 (PB9), U3.4 (SDA)
- net SAI_FS: now also U13.C3 (PE4)
- net SAI_SCK: now also IC1.21 (PB10), U13.D3 (PE5); no longer IC1.29 (PA8)
- net SAI_SD: now also U13.C6 (PD6)
- net SPI_MISO: now also U13.A6 (PB4(NJTRST))
- net SPI_MOSI: now also U13.D6 (PD7)
- net SPI_SCK: now also U13.A7 (PB3(JTDO)
- net USB_DP: now also U2.13 (DP)
- net VBUS: now also R14.2, U3.13 (ISN); no longer C18.2, R7.2
- net VBUS_EN: now also IC1.2 (PC13); no longer IC1.5 (PH0)
- net VBUS_SW: now also IC1.3 (PC14), R33.2; no longer IC1.6 (PH1), R8.2
- net at R21.2, R22.1: now also U12.6 (ADJ-); no longer C64.2
- net DSP_MCK: now reaches IC2.21 (XTALIN/MCLK)
- net DSP_MCK: no longer C29.2
- net at IC2.22 (XTALOUT): no longer R13.2
- net at R16.1, U9.3 (+): now also IC3.20 (OUT2)
- net at C53.3: now also U8.5 (V+); no longer U9.5 (V+)
- net at R20.1: now also C56.1, U11.7 (SET); no longer C45.1
- net at C72.1: now also L2.1, U3.8 (SW1); no longer R25.1
- net +5V: now reaches C3.1, C4.1, C5.1, L1.2, U7.1 (IN1), U7.18 (SS_CTRL1), U7.2 (IN1), U7.4 (IN2), U7.5 (IN1), U7.8 (SS_CTRL2)
- net +5V: now also C16.1, C30.2, C45.1, R1.2, R2.1, C91.1, C92.1, C93.1, C94.1, U11.1 (IN), U11.2 (IN), U15.1 (IN1), U15.18 (SS_CTRL1), U15.2 (IN1), U15.4 (IN2), U15.5 (IN1), U15.8 (SS_CTRL2), U2.16 (VBAT), U3.18 (VCC); no longer R1.1, R4.2
- net 5V_GOOD: now reaches U7.20 (EN1), U7.6 (EN2)
- net 5V_GOOD: no longer R4.1, U1.5 (PG)
- net at C17.1: now also U2.2 (CLKOUT), U2.23 (VDD18); no longer R6.2
- net at C3.2, U1.3 (FB): now also R2.2, R4.1; no longer R1.2, R2.1
- net at C62.2: now also U12.1 (CBST-)
- net Earth: now reaches R26.2
- net Earth: now also C1.2, C10.2, C11.2, C12.2, C13.1, C14.2, C16.2, C17.2, C18.2, C20.2, C21.2, C22.2, C23.2, C24.2, C25.2, C26.2, C27.2, C29.2, C30.1, C32.2, C33.2, C34.2, C35.2, C36.2, C37.2, C38.2, C39.2, C4.2, C40.2, C41.2, C42.2, C43.2, C44.2, C45.2, C46.2, C47.2, C48.2, C5.2, C50.2, C53.2, C54.2, C56.2, C57.2, C58.2, C59.2, C6.2, C61.2, C63.2, C65.2, C66.1, C67.2, C68.2, C7.2, C71.1, C76.2, C79.2, C80.2, C81.2, C82.2, D3.2 (A2), IC1.23 (VSS), IC1.35 (VSS), IC1.47 (VSS), IC1.49 (VSS), IC1.8 (VSSA), IC2.1 (DGND), IC2.14 (PGND), IC2.17 (DGND), IC2.19 (DGND), IC2.25 (DGND), IC2.3 (VDRIVE), IC2.36 (DGND), IC2.37 (DGND), IC2.54 (DGND), IC2.55 (DGND), IC2.6 (AGND), IC2.72 (DGND), IC2.73 (EP), J1.A1 (GND), J1.A12 (GND), J1.B1 (GND), J1.B12 (GND), J1.S1 (SHIELD), R11.1, R13.2, R18.2, R19.2, R20.2, R21.1, R23.2, R25.2, R29.2, R30.1, R32.2, R4.2, R6.2, R7.2, R8.2, SW1.1 (A), U1.4 (COMP), U1.8 (GND), U10.2 (GND), U17.4 (COMP), U17.8 (GND), U4.2, U5.10 (NC), U5.11 (NC), U5.12 (NC), U5.13 (VSS), U5.14 (NC), U5.16 (NC), U5.4 (NC), U5.8 (NC), U5.9 (NC), U7.13 (GND), U7.25 (GND), U7.3 (GND), U8.2 (GND), U9.2 (GND), C106.2, C15.2, C52.2, C55.2, C69.1, C70.2, C75.2, C77.2, C83.2, C84.2, C85.2, C86.2, C89.2, C90.2, C91.2, C92.2, C93.2, C94.2, C95.2, C96.2, C97.2, D1.1 (A1), D2.2 (A), IC3.14 (SENSE2), IC3.15 (GND), IC3.16 (GND), IC3.17 (SENSE1), IC3.5 (GND), IC3.6 (GND), J2.1 (Pin_1), J2.2 (Pin_2), R37.2, R39.2, U11.11 (GND), U11.8 (GND), U12.12 (RT), U12.14 (MODE), U12.19 (GND), U14.3 (GND), U15.13 (GND), U15.25 (GND), U15.3 (GND), U2.17 (VBUS), U2.25 (GND), U3.17 (AGND), U3.2 (MODE), U3.21 (EXTVCC), U3.9 (PGND), Y2.2, Y2.4; no longer R27.1
- net at D4.1 (K), D5.2 (A): now also C51.2; no longer C51.1
- net at R15.1, U8.3 (+): now also IC3.1 (OUT1)
- net at R17.1, U10.3 (+): now also IC3.10 (OUT3)
- net at J1.A4 (VBUS), J1.A9 (VBUS), J1.B4 (VBUS)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: now also D1.2 (A2), D2.1 (K), D6.1 (K); no longer U4.5
- net at C18.1: now also U2.15 (VDD33), U2.18 (ID); no longer R7.1
- net at C54.3: now also U9.5 (V+); no longer U10.5 (V+)
- net at R19.1: now also U11.5 (ILIM)
- net at D5.1 (K): now also C49.1, IC3.13 (VBOOT); no longer C49.2
- net +12V: now reaches C63.1
- net +12V: now also C1.1, U1.1 (VIN), U1.2 (EN), U12.13 (EN+), U12.3 (VIN+), U12.4 (EN-)
- net at R13.1: now also C74.2; no longer C30.2
- net at R8.1: now also U2.19 (RBIAS); no longer U4.1
- net at R9.2: now also U13.D5 (BOOT0); no longer IC1.44 (PH3)
- net +15V: no longer names the net of C67.1
- net +15V: now also U12.11 (VIN-), U12.18 (VOUT+)
- removed net GND1: C1.2, C10.2, C11.2, C12.2, C13.2, C16.2, C17.2, C19.1, C20.2, C21.2, C22.2, C23.2, C24.2, C25.2, C26.2, C27.2, C29.1, C30.1, C32.2, C33.2, C34.2, C35.2, C36.2, C37.2, C38.2, C39.2, C4.2, C40.2, C41.2, C42.2, C43.2, C44.2, C45.2, C46.2, C47.2, C48.2, C5.2, C50.2, C53.2, C54.2, C56.2, C57.2, C58.2, C59.2, C6.2, C68.2, C7.2, C76.2, C79.2, C80.2, C81.2, C82.2, D3.2 (A2), IC1.23 (VSS), IC1.35 (VSS), IC1.47 (VSS), IC1.49 (VSS), IC1.8 (VSSA), IC2.1 (DGND), IC2.14 (PGND), IC2.17 (DGND), IC2.19 (DGND), IC2.25 (DGND), IC2.3 (VDRIVE), IC2.36 (DGND), IC2.37 (DGND), IC2.54 (DGND), IC2.55 (DGND), IC2.6 (AGND), IC2.72 (DGND), IC2.73 (EP), J1.A1 (GND), J1.A12 (GND), J1.B1 (GND), J1.B12 (GND), J1.S1 (SHIELD), R11.1, R19.2, R2.2, R20.2, R23.2, R29.2, R30.1, R32.2, R5.2, SW1.1 (A), U1.4 (COMP), U1.8 (GND), U10.2 (GND), U17.4 (COMP), U17.8 (GND), U4.2, U5.10 (NC), U5.11 (NC), U5.12 (NC), U5.13 (VSS), U5.14 (NC), U5.16 (NC), U5.4 (NC), U5.8 (NC), U5.9 (NC), U7.13 (GND), U7.25 (GND), U7.3 (GND), U8.2 (GND), U9.2 (GND)
- removed net GND2: C61.2, C62.1, C65.2, C66.2, C67.2, C71.2, C72.2, C73.2, R22.2, R24.2, R25.2, R27.2
- net VDD_OK renamed DIGI_EN
- net DIGI_EN: no longer C19.2, IC1.7 (NRST)
- removed net VIR: C64.1, C65.1, C66.1, C71.1, R21.1, R3.2
- net VIR_OK renamed OA_V+
- net OA_V+: now also C70.1, U12.17 (LDO+)
- new net: C77.1, C83.1, C84.1, C95.1, C96.1, C97.1, R14.1, U3.11 (VOUT), U3.12 (ISP)
- new net: C73.1, L2.2, U3.10 (SW2)
- new net: C73.2, U3.19 (BOOT2)
- new net: C87.2, R36.2, R37.1, U15.10 (FB2)
- new net: C88.2, R38.2, R39.1, U15.16 (FB1)
- new net: D6.2 (A), U4.5
- new net: R18.1, R3.2, U12.16 (ADJ+)
- new net: C72.2, U3.20 (BOOT1)
- new net: C50.1, IC3.11 (VREF)
- new net: C51.1, IC3.12 (VCP)
- new net: C15.1, U2.9 (VDDIO)
- new net: U13.C1 (PH0), Y2.1
- new net: U13.C2 (VSS), U13.E4 (VSS), U13.E5 (VSS), U13.E6 (VSS), U13.J1 (VSS)
- new net: U13.D1 (PH1), Y2.3
- new net: C19.2, U13.E1 (NRST)
- new net: R7.1, U3.6 (FSW)
- new net: C64.1, U12.10 (CINV+)
- new net: C64.2, U12.9 (CINV-)
- new net: R33.1, U4.1
- new net: C55.3, U10.5 (V+)
- new net: R5.2, R6.1, U3.1 (EN_UVLO)
- new net: C74.1, C75.1, U3.15 (COMP)
- new net: C29.1, U3.5 (DITH_SYNC)
- new net: C69.2, U12.8 (VOUT-)
- new net: C65.1, U12.15 (BYP+)
- new net: C62.1, U12.2 (CBST+)
- new net: C66.2, U12.5 (BYP-)
- new net: R24.2, R25.1, U11.6 (PGFB)
- new net: C85.1, U15.19 (NR/SS1)
- new net: C86.1, U15.7 (NR/SS2)
- new net 5V_OK: R1.1, U1.5 (PG), U11.3 (EN/UV), U14.1, U15.20 (EN1), U15.6 (EN2)
- new net DAC_*MUTE: R26.1, U14.2
- new net DAC_DVDD: C88.1, C89.1, R38.1, U15.14 (OUT1), U15.15 (OUT1)
- new net OA_V-: C71.2, R22.2, U12.7 (LDO-)
- new net ULPI_D0: U13.K2 (PA3), U2.4 (DATA0)
- new net ULPI_D1: U13.J4 (PB0), U2.5 (DATA1)
- new net ULPI_D2: U13.K4 (PB1), U2.6 (DATA2)
- new net ULPI_D3: U13.J7 (PB10), U2.7 (DATA3)
- new net ULPI_D4: U13.K7 (PB11), U2.8 (DATA4)
- new net ULPI_D5: U13.K8 (PB12), U2.10 (DATA5)
- new net ULPI_D6: U13.J8 (PB13), U2.11 (DATA6)
- new net ULPI_D7: U13.C5 (PB5), U2.12 (DATA7)
- new net ULPI_DIR: U13.E2 (PC2_C), U2.1 (DIR)
- new net ULPI_NXT: U13.F3 (PC3_C), U2.3 (NXT)
- new net ULPI_STP: U13.F1 (PC0), U2.24 (STP)
- new net USB_CK: U13.H3 (PA5), U2.21 (REFCLK/XI)
- new net USB_DM: U2.14 (DM)
- new net USB_EN: U2.22 (~{RESETB})
- new net USB_SOF: IC1.29 (PA8)
Other:
- note added: "5V Power Supply"
- note added: "DAC Analog Power Supply"
- note added: "DAC Digital Power Supply"
- note added: "Op-Amp Power Supply (+/-15V)"
- note added: "USB 2.0 HS PHY"
- note added: "USB-C"
- note removed: "Inputs"
- note removed: "Isolated DC Power Supply"
- note removed: "Isolated Regulator"
- moved on the sheet: C20, C21, C22, C23, C24, C25, C26, C27, C28, C31, C32, C33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
